Commit message: change urdf dof_pos, add init_joint_angle

File: assets/urdf/nz/urdf/nz.urdf (robot description, URDF)
Before this commit: robot nz, 11 links, 10 joints
Links:
- link left_calf_link: mass 0.6553 -> 0.8053
- link left_hip_link: mass 3.3424287 -> 3.3489287
- link left_thigh_link: mass 0.4141741 -> 0.43777
- link right_calf_link: mass 0.6553 -> 0.8053
- link right_hip_link: mass 3.3276491 -> 3.3496969
- link right_thigh_link: mass 0.2639971 -> 0.43777
Joints:
- joint left_calf_joint: limit lower=0 upper=1.3963 effort=40 velocity=0 -> lower=-1.3963 upper=0 effort=40 velocity=0; origin xyz=-0.15513 0.018 -0.091296 rpy=0 0 0 -> xyz=-0.074709 0.018 -0.16376 rpy=0 0 0
- joint left_hip_joint: axis 1 0 0 -> 0 0 0; origin xyz=0.151248020480631 0.103301979532171 0.0740000350635592 rpy=-0.000730179484732082 0 0 -> xyz=0.15125 0.1033 0.074 rpy=-0.00073018 0 0
- joint left_knee_wheel_joint: origin xyz=-0.048296 0.02265 0.012941 rpy=0 0 0 -> xyz=-0.048296 0.02265 -0.012941 rpy=0 0 0
- joint left_wheel_joint: origin xyz=0.20864 0.027 -0.055905 rpy=0 0 0 -> xyz=0.20864 0.027 0.055905 rpy=0 0 0
- joint right_calf_joint: limit lower=0 upper=1.3963 effort=40 velocity=0 -> lower=-1.3963 upper=0 effort=40 velocity=0; origin xyz=-0.15513 -0.018001 -0.091296 rpy=0 0 0 -> xyz=-0.074709 -0.018 -0.16376 rpy=0 0 0
- joint right_hip_joint: axis 1 0 0 -> 0 0 0
- joint right_knee_wheel_joint: origin xyz=-0.0482962913144536 -0.0226499999999995 0.0129409522551254 rpy=0 0 0 -> xyz=-0.048296 -0.02265 -0.012941 rpy=0 0 0
- joint right_wheel_joint: origin xyz=0.20864 -0.026999 -0.055905 rpy=0 0 0 -> xyz=0.20864 -0.027 0.055905 rpy=0 0 0
